File: kicad/kicad-workshop.kicad_pcb (KiCad board)
At the start: 2 copper layers, 40 x 18.5 mm, 21 parts, among them J1 TYPE-C-31-M-12, J2 Conn_01x04, J3 Conn_01x04, SW2 PEC12R-4130F-S0012, U1 EFM32HG309F64G-B-QFN24

Commit message: change LED to single color The 1x1 mm LED was too difficult for assembly, mostly locating pin 1
Parts:
- removed R8, R9: 240, kicad-workshop:R_0603_1608Metric
- D1: value UHD1110-FKA -> LED; footprint kicad_pcb:LED_cree_4_1x1 -> LED_SMD:LED_0603_1608Metric
- moved D1 1.53 mm to (163.7, 83.3), turned to 0 degrees
Connections:
- net /R renamed /LED
- D1 pad 1: Net-(D1-Pad1) -> GND
- R7 pad 1: Net-(D1-Pad3) -> Net-(D1-Pad2)
- U1 pad 6: /G -> Net-(U1-Pad6)
- U1 pad 8: /B -> Net-(U1-Pad8)
Routing:
- net /VBUS: track 25.0 -> 14.0 mm
- net /G: track 2.86 -> 0.00 mm
- net Net-(D1-Pad3): track 2.48 -> 0.00 mm
- net /B: track 1.61 -> 0.00 mm
- net Net-(D1-Pad1): track 1.29 -> 0.00 mm
- net GND: track 6.73 -> 7.64 mm, vias 8 -> 9
